File: PCB/attiny.kicad_pcb (KiCad board)
At the start: 2 copper layers, 53.3 x 25.4 mm, 33 parts, among them J1 Conn_01x04, J2 Conn_01x04, J3 Conn_01x02, Q1 BC817, Q2 Q_Photo_NPN, SW1 SW_SPST, U1 ATtiny814-SS

Commit message: add logo 5dn1L
Parts:
- added G***: LOGO, ensylam:5dn1l, B.Cu at (137.2, 68.6)
